Commit message: Update launch for single FR3

File: crisp_controllers_robot_demos/config/fr3/fr3.ros2_control.urdf.xacro (robot description, xacro)
@@ -13,4 +13,5 @@
              robot_ip
              use_fake_hardware
+             enable_mujoco_gui
              arm_prefix:=''">
     <xacro:property name="arm_prefix_modified" value="${'' if arm_prefix == '' else arm_prefix + '_'}" />
@@ -27,4 +28,5 @@
             <plugin>crisp_mujoco_sim/Simulator</plugin>
             <param name="mujoco_model">$(find crisp_controllers_robot_demos)/config/fr3/scene.xml</param>
+            <param name="enable_gui">${enable_mujoco_gui}</param>
           </xacro:if>
         </hardware>

File: crisp_controllers_robot_demos/config/fr3/fr3.urdf.xacro (robot description, xacro)
@@ -3,8 +3,9 @@
   <xacro:include filename="$(find franka_description)/robots/common/franka_robot.xacro"/>
   <xacro:include filename="$(find crisp_controllers_robot_demos)/config/fr3/fr3.ros2_control.urdf.xacro"/>
-  <xacro:macro name="fr3"
+<xacro:macro name="fr3"
          params="arm_id
              robot_ip
              use_fake_hardware
+             enable_mujoco_gui:=false
              arm_prefix:=''
              hand:=true
@@ -40,4 +41,5 @@
             robot_ip="${robot_ip}"
             use_fake_hardware="$(arg use_fake_hardware)"
+            enable_mujoco_gui="${enable_mujoco_gui}"
             arm_prefix="${arm_prefix}"/>
   </xacro:macro>

File: crisp_controllers_robot_demos/config/fr3/fr3_dual.urdf.xacro (robot description, xacro)
@@ -8,4 +8,5 @@
   <!-- Should a fake hardware be used? -->
   <xacro:arg name="use_fake_hardware" default="true" />
+  <xacro:arg name="enable_mujoco_gui" default="false" />
   <!-- Should fake sensors be used? -->
   <xacro:arg name="fake_sensor_commands" default="false" />
@@ -16,4 +17,5 @@
     robot_ip="$(arg robot_ip_left)"
     use_fake_hardware="$(arg use_fake_hardware)"
+    enable_mujoco_gui="$(arg enable_mujoco_gui)"
     hand="$(arg hand)"
     arm_prefix="left"
@@ -23,4 +25,5 @@
     robot_ip="$(arg robot_ip_right)"
     use_fake_hardware="$(arg use_fake_hardware)"
+    enable_mujoco_gui="$(arg enable_mujoco_gui)"
     hand="$(arg hand)"
     arm_prefix="right"

File: crisp_controllers_robot_demos/config/fr3/fr3_single.urdf.xacro (robot description, xacro)
@@ -15,4 +15,5 @@
   <!-- Should a fake hardware be used? -->
   <xacro:arg name="use_fake_hardware" default="false" />
+  <xacro:arg name="enable_mujoco_gui" default="false" />
   <!-- Should fake sensors be used? -->
   <xacro:arg name="fake_sensor_commands" default="false" />
@@ -30,4 +31,5 @@
     robot_ip="$(arg robot_ip)"
     use_fake_hardware="$(arg use_fake_hardware)"
+    enable_mujoco_gui="$(arg enable_mujoco_gui)"
     arm_prefix="$(arg arm_prefix)"
     hand="$(arg load_gripper)"
