Commit message: update body in unified kinematic file for urdf and xml

File: crisp_controllers_robot_demos/config/fr3/fr3_dual.urdf.xacro (robot description, xacro)
@@ -26,13 +26,50 @@
     arm_prefix="right"
   />
+  <!-- World link -->
   <link name="world"/>
-  <!-- Define the transform between both arms -->
-  <joint name="left_base_to_world_joint" type="fixed"> <parent link="world"/>
+  <!-- Base platform link with Duo Franka Base mesh -->
+  <link name="base_link">
+    <visual>
+      <origin xyz="0 0 0" rpy="0 0 0"/>
+      <geometry>
+        <mesh filename="package://crisp_controllers_robot_demos/config/fr3/assets/body/Duo_Franka_Base.stl"/>
+      </geometry>
+      <material name="gray">
+        <color rgba="0.5 0.5 0.5 1"/>
+      </material>
+    </visual>
+    <collision>
+      <origin xyz="0 0 0" rpy="0 0 0"/>
+      <geometry>
+        <mesh filename="package://crisp_controllers_robot_demos/config/fr3/assets/body/Duo_Franka_Base.stl"/>
+      </geometry>
+    </collision>
+    <inertial>
+      <origin xyz="0 0 0" rpy="0 0 0"/>
+      <mass value="10.0"/>
+      <inertia ixx="0.1" ixy="0" ixz="0" iyy="0.1" iyz="0" izz="0.1"/>
+    </inertial>
+  </link>
+  <!-- Fix base platform to world -->
+  <joint name="world_to_base_joint" type="fixed">
+    <parent link="world"/>
+    <child link="base_link"/>
+    <origin xyz="0 0 0" rpy="0 0 0"/>
+  </joint>
+  <!-- Mount left arm on base platform -->
+  <!-- MuJoCo: pos="0.056 0.119324 0.194376" quat="0.9239 -0.3827 0 0" -->
+  <!-- Quaternion [0.9239, -0.3827, 0, 0] converts to RPY [-0.785398, 0, 0] (approx -45 deg roll) -->
+  <joint name="left_base_to_base_joint" type="fixed">
+    <parent link="base_link"/>
     <child link="left_base"/>
-    <origin rpy="0 0 0" xyz="0 0 0"/>
+    <origin xyz="0.056 0.119324 0.194376" rpy="-0.785398 0 0"/>
   </joint>
-  <joint name="right_base_to_world_joint" type="fixed"> <parent link="world"/>
+  <!-- Mount right arm on base platform -->
+  <!-- MuJoCo: pos="0.056 -0.119324 0.194376" quat="0.9239 0.3827 0 0" -->
+  <!-- Quaternion [0.9239, 0.3827, 0, 0] converts to RPY [0.785398, 0, 0] (approx +45 deg roll) -->
+  <joint name="right_base_to_base_joint" type="fixed">
+    <parent link="base_link"/>
     <child link="right_base"/>
-    <origin rpy="0 0 0" xyz="0 1.0 0"/>
+    <origin xyz="0.056 -0.119324 0.194376" rpy="0.785398 0 0"/>
   </joint>
 </robot>

Commit message: refactor: create 2 demo urdf for dual Franka setup

File: crisp_controllers_robot_demos/config/fr3/fr3_dual.urdf.xacro (robot description, xacro)
@@ -26,50 +26,13 @@
     arm_prefix="right"
   />
-  <!-- World link -->
   <link name="world"/>
-  <!-- Base platform link with Duo Franka Base mesh -->
-  <link name="base_link">
-    <visual>
-      <origin xyz="0 0 0" rpy="0 0 0"/>
-      <geometry>
-        <mesh filename="package://crisp_controllers_robot_demos/config/fr3/assets/body/Duo_Franka_Base.stl"/>
-      </geometry>
-      <material name="gray">
-        <color rgba="0.5 0.5 0.5 1"/>
-      </material>
-    </visual>
-    <collision>
-      <origin xyz="0 0 0" rpy="0 0 0"/>
-      <geometry>
-        <mesh filename="package://crisp_controllers_robot_demos/config/fr3/assets/body/Duo_Franka_Base.stl"/>
-      </geometry>
-    </collision>
-    <inertial>
-      <origin xyz="0 0 0" rpy="0 0 0"/>
-      <mass value="10.0"/>
-      <inertia ixx="0.1" ixy="0" ixz="0" iyy="0.1" iyz="0" izz="0.1"/>
-    </inertial>
-  </link>
-  <!-- Fix base platform to world -->
-  <joint name="world_to_base_joint" type="fixed">
-    <parent link="world"/>
-    <child link="base_link"/>
-    <origin xyz="0 0 0" rpy="0 0 0"/>
+  <!-- Define the transform between both arms -->
+  <joint name="left_base_to_world_joint" type="fixed"> <parent link="world"/>
+    <child link="left_base"/>
+    <origin rpy="0 0 0" xyz="0 0 0"/>
   </joint>
-  <!-- Mount left arm on base platform -->
-  <!-- MuJoCo: pos="0.056 0.119324 0.194376" quat="0.9239 -0.3827 0 0" -->
-  <!-- Quaternion [0.9239, -0.3827, 0, 0] converts to RPY [-0.785398, 0, 0] (approx -45 deg roll) -->
-  <joint name="left_base_to_base_joint" type="fixed">
-    <parent link="base_link"/>
-    <child link="left_base"/>
-    <origin xyz="0.056 0.119324 0.194376" rpy="-0.785398 0 0"/>
-  </joint>
-  <!-- Mount right arm on base platform -->
-  <!-- MuJoCo: pos="0.056 -0.119324 0.194376" quat="0.9239 0.3827 0 0" -->
-  <!-- Quaternion [0.9239, 0.3827, 0, 0] converts to RPY [0.785398, 0, 0] (approx +45 deg roll) -->
-  <joint name="right_base_to_base_joint" type="fixed">
-    <parent link="base_link"/>
+  <joint name="right_base_to_world_joint" type="fixed"> <parent link="world"/>
     <child link="right_base"/>
-    <origin xyz="0.056 -0.119324 0.194376" rpy="0.785398 0 0"/>
+    <origin rpy="0 0 0" xyz="0 1.0 0"/>
   </joint>
 </robot>
